Commit message: fix typo

File: GRX/GR1/GR1T2/URDF/urdf/GR1T2_upper.urdf (robot description, URDF)
Before this commit: robot GR1T2_upper, 37 links, 36 joints
Joints:
- joint l_hip_yaw: type joint -> fixed

Commit message: fix typo

File: GRX/GR1/GR1T2/URDF/urdf/GR1T2_upper.urdf (robot description, URDF)
Before this commit: robot GR1T2_upper, 37 links, 36 joints
Joints:
- joint waist_roll: type  -> revolute
